Commit message: feat(sim): add initial Gazebo simulation definitions

File: src/robot_package/description/robot.urdf.xacro (robot description, xacro)
@@ -2,3 +2,4 @@
 <robot xmlns:xacro="https://www.ros.org/wiki/xacro" name="robot">
     <xacro:include filename="robot_core.xacro" />
+    <xacro:include filename="gazebo_control.xacro"/>
 </robot>

File: src/robot_package/description/robot_core.xacro (robot description, xacro)
@@ -14,4 +14,5 @@
     <xacro:property name="wheel_length" value="0.024"/>
     <xacro:property name="wheel_mass" value="0.03"/>
+    <xacro:property name="max_steer_angle" value="0.52"/> <!-- 30 Degrees turning radius -->
     <!-- Joint offsets -->
     <xacro:property name="track_width" value="0.158"/>
@@ -42,5 +43,5 @@
         </collision>
         <xacro:inertial_box mass="${chassis_mass}" x="${chassis_length}" y="${chassis_width}" z="${chassis_height}">
-            <origin xyz="$0 0 0"/>
+            <origin xyz="0 0 0"/>
         </xacro:inertial_box>
     </link>

File: src/robot_package/description/wheel_macros.xacro (robot description, xacro)
@@ -26,5 +26,12 @@
             </xacro:inertial_cylinder>
         </link>
-        </xacro:macro>
+        <!-- Tire Friction -->
+        <gazebo reference="${prefix}_wheel_link">
+            <mu1>0.9</mu1>
+            <mu2>0.9</mu2>
+            <kp>100000000.0</kp>
+            <kd>1.0</kd>
+        </gazebo>
+    </xacro:macro>
     <!-- Steered Wheel Macro -->
      <xacro:macro name="steered_wheel" params="prefix x_offset y_reflect">
@@ -35,7 +42,11 @@
             <origin xyz="${x_offset} ${y_reflect * wheel_offset_y} 0"/>
             <axis xyz="0 0 1"/>
-            <limit lower="-0.52" upper="0.52" effort="10.0" velocity="5.0"/>
+            <limit lower="-${max_steer_angle}" upper="${max_steer_angle}" effort="10.0" velocity="5.0"/>
         </joint>
+        <!-- Steering Knuckle Inertial Tag for simulation -->
         <link name="${prefix}_steer_link">
+            <xacro:inertial_box mass="0.01" x="0.02" y="0.02" z="0.02">
+                <origin xyz="0 0 0"/>
+            </xacro:inertial_box>
         </link>
         <!-- Wheel -->
@@ -62,4 +73,10 @@
             </xacro:inertial_cylinder>
         </link>
+        <gazebo reference="${prefix}_wheel_link">
+            <mu1>0.9</mu1>
+            <mu2>0.9</mu2>
+            <kp>100000000.0</kp>
+            <kd>1.0</kd>
+        </gazebo>
      </xacro:macro>
 </robot>
