File: hardware/schematics/vetronics/vetronics.kicad_sch (KiCad schematic)
At the start: 11 parts, among them SW1 12V 15A SPST Toggle

Commit message: hardware: added mechanical components
hw(vetronics): fixed electronic inconsistency with the rplidar in the schematic
Parts:
- J_ESC_PWR: value QuicRun 1060 Input (Deans) -> QuicRun 1060 Input
- U_HUB1: symbol Connector:Conn_01x03_Pin -> Connector:Conn_01x04_Pin
- U_SENS1: symbol Connector:Conn_01x03_Pin -> Connector:Conn_01x01_Pin
Connections:
- net +5V: no longer U_SENS1.1 (Pin_1)
- net GND: no longer U_SENS1.2 (Pin_2)
- net USB_DATA_HUB: no longer U_SENS1.3 (Pin_3)
- new net USB_LIDAR: U_HUB1.4 (Pin_4), U_SENS1.1 (Pin_1)
Other:
- title: Project POLEMARCHUS - Vehicle Avionics & Power Distribution -> Project POLEMARCHUS - Vetronics & Power Distribution
