Commit message: feat(sim): added visual meshes and automated ROS 2 Gazebo bridge

File: src/tamiya_rover_description/description/robot_core.xacro (robot description, xacro)
@@ -16,8 +16,9 @@
     <xacro:property name="max_steer_angle" value="0.52"/> <!-- 30 Degrees turning radius -->
     <!-- Joint offsets -->
-    <xacro:property name="track_width" value="0.158"/>
+    <xacro:property name="track_width" value="0.182"/>
     <xacro:property name="wheel_base" value="0.257"/>
     <!-- Calculated Joint origins -->
     <xacro:property name="wheel_offset_y" value="${track_width / 2}"/>
+    <xacro:property name="wheel_offset_z" value="${chassis_height / 2}"/>
     <!-- Rear wheels are at x=0. Front wheels are at x=wheel_base -->
     <!-- Base Link -->
@@ -33,6 +34,7 @@
         <visual>
             <geometry>
-                <box size="${chassis_length} ${chassis_width} ${chassis_height}"/>
+                <mesh filename="file://$(find tamiya_rover_description)/meshes/tt02d_chassis.stl" scale="0.001 0.001 0.001"/>
             </geometry>
+            <origin xyz="0 0 0" rpy="0 0 0"/>
             <material name="gray"/>
         </visual>
@@ -46,4 +48,20 @@
         </xacro:inertial_box>
     </link>
+    <!-- Vetronics Deck Link -->
+    <joint  name="vetronics_deck_joint" type="fixed">
+        <parent link="chassis_link"/>
+        <child link="vetronics_deck_link"/>
+        <!-- z-offset to place it on top of the chassis -->
+        <origin xyz="0 0 ${chassis_height / 2 + 0.011}" rpy="0 0 0"/>
+    </joint>
+    <link name="vetronics_deck_link">
+        <visual>
+            <geometry>
+                <mesh filename="file://$(find tamiya_rover_description)/meshes/vetronics_deck.stl" scale="0.001 0.001 0.001"/>
+            </geometry>
+            <origin xyz="0 0 0" rpy="0 0 0"/>
+            <material name="gray"/>
+        </visual>
+    </link>
     <!-- Rear Right Wheel Link -->
     <xacro:fixed_wheel prefix="rr" x_offset="0" y_reflect="-1" />

File: src/tamiya_rover_description/description/robot_materials.xacro (robot description, xacro)
@@ -2,8 +2,8 @@
 <robot xmlns:xacro="http://www.ros.org/wiki/xacro" >
     <material name="gray">
-        <color rgba="0.5 0.5 0.5 1" />
+        <color rgba="0.6 0.6 0.6 1" />
     </material>
     <material name="black">
-        <color rgba="0 0 0 1"/>
+        <color rgba="0.1 0.1 0.1 1"/>
     </material>
 </robot>

File: src/tamiya_rover_description/description/wheel_macros.xacro (robot description, xacro)
@@ -6,12 +6,14 @@
             <parent link="base_link"/>
             <child link="${prefix}_wheel_link"/>
-            <origin xyz="${x_offset} ${y_reflect * wheel_offset_y} 0" rpy="-${pi / 2} 0 0"/>
-            <axis xyz="0 0 1"/>
+            <origin xyz="${x_offset} ${y_reflect * wheel_offset_y} ${wheel_offset_z}" rpy="0 0 0"/>
+            <axis xyz="0 1 0"/>
         </joint>
         <link name="${prefix}_wheel_link">
             <visual>
                 <geometry>
-                    <cylinder radius="${wheel_radius}" length="${wheel_length}"/>
+                    <mesh filename="file://$(find tamiya_rover_description)/meshes/tt02d_wheel.stl" scale="0.001 0.001 0.001"/>
                 </geometry>
+                <!-- Dinamically flip the mesh -->
+                <origin xyz="0 0 0" rpy="0 0 ${(1 - y_reflect) / 2 * pi}"/>
                 <material name="black"/>
             </visual>
@@ -20,4 +22,5 @@
                     <cylinder radius="${wheel_radius}" length="${wheel_length}"/>
                 </geometry>
+                <origin xyz="0 0 0" rpy="-${pi / 2} 0 0"/>
                 <material name="black"/>
             </collision>
@@ -40,5 +43,5 @@
             <parent link="base_link"/>
             <child link="${prefix}_steer_link"/>
-            <origin xyz="${x_offset} ${y_reflect * wheel_offset_y} 0"/>
+            <origin xyz="${x_offset} ${y_reflect * wheel_offset_y} ${wheel_offset_z}"/>
             <axis xyz="0 0 1"/>
             <limit lower="-${max_steer_angle}" upper="${max_steer_angle}" effort="10.0" velocity="5.0"/>
@@ -54,12 +57,14 @@
             <parent link="${prefix}_steer_link"/>
             <child link="${prefix}_wheel_link"/>
-            <origin xyz="0 0 0" rpy="-${pi / 2} 0 0"/>
-            <axis xyz="0 0 1"/>
+            <origin xyz="0 0 0" rpy="0 0 0"/>
+            <axis xyz="0 1 0"/>
         </joint>
         <link name="${prefix}_wheel_link">
             <visual>
                 <geometry>
-                    <cylinder radius="${wheel_radius}" length="${wheel_length}"/>
+                    <mesh filename="file://$(find tamiya_rover_description)/meshes/tt02d_wheel.stl" scale="0.001 0.001 0.001"/>
                 </geometry>
+                <!-- Dinamically flip the mesh -->
+                <origin xyz="0 0 0" rpy="0 0 ${(1 - y_reflect) / 2 * pi}"/>
                 <material name="black"/>
             </visual>
@@ -68,4 +73,5 @@
                     <cylinder radius="${wheel_radius}" length="${wheel_length}"/>
                 </geometry>
+                <origin xyz="0 0 0" rpy="-${pi / 2} 0 0"/>
             </collision>
             <xacro:inertial_cylinder mass="${wheel_mass}" length="${wheel_length}" radius="${wheel_radius}">

Commit message: fix: made meshes paths relative to the package for visualization over ssh

File: src/tamiya_rover_description/description/robot_core.xacro (robot description, xacro)
@@ -34,5 +34,5 @@
         <visual>
             <geometry>
-                <mesh filename="file://$(find tamiya_rover_description)/meshes/tt02d_chassis.stl" scale="0.001 0.001 0.001"/>
+                <mesh filename="package://tamiya_rover_description/meshes/tt02d_chassis.stl" scale="0.001 0.001 0.001"/>
             </geometry>
             <origin xyz="0 0 0" rpy="0 0 0"/>
@@ -58,5 +58,5 @@
         <visual>
             <geometry>
-                <mesh filename="file://$(find tamiya_rover_description)/meshes/vetronics_deck.stl" scale="0.001 0.001 0.001"/>
+                <mesh filename="package://tamiya_rover_description/meshes/vetronics_deck.stl" scale="0.001 0.001 0.001"/>
             </geometry>
             <origin xyz="0 0 0" rpy="0 0 0"/>

File: src/tamiya_rover_description/description/wheel_macros.xacro (robot description, xacro)
@@ -12,5 +12,5 @@
             <visual>
                 <geometry>
-                    <mesh filename="file://$(find tamiya_rover_description)/meshes/tt02d_wheel.stl" scale="0.001 0.001 0.001"/>
+                    <mesh filename="package://tamiya_rover_description/meshes/tt02d_wheel.stl" scale="0.001 0.001 0.001"/>
                 </geometry>
                 <!-- Dinamically flip the mesh -->
@@ -63,5 +63,5 @@
             <visual>
                 <geometry>
-                    <mesh filename="file://$(find tamiya_rover_description)/meshes/tt02d_wheel.stl" scale="0.001 0.001 0.001"/>
+                    <mesh filename="package://tamiya_rover_description/meshes/tt02d_wheel.stl" scale="0.001 0.001 0.001"/>
                 </geometry>
                 <!-- Dinamically flip the mesh -->
