Commit message: fix: fixed lidar orientation in robot_description

File: src/tamiya_rover_description/description/lidar.xacro (robot description, xacro)
@@ -6,5 +6,5 @@
         <parent link="vetronics_deck_link"/>
         <child link="laser_frame"/>
-        <origin xyz="0.033 0 0.070" rpy="0 0 0"/>
+        <origin xyz="0.033 0 0.070" rpy="0 0 ${pi}"/>
     </joint>
     <link name="laser_frame">
